File: MBot.kicad_pcb (KiCad board)
At the start: 4 copper layers, 60 x 60 mm, 111 parts, among them J1 Micro_SD_Card_Det1, J10 Conn_01x04, J11 Conn_01x06, J12 Conn_01x04, J14 Conn_01x04, J16 Conn_01x06, J2 Barrel_Jack_Switch_Pin3Ring, J3 Screw_Terminal_01x02, J4 Conn_01x03, J5 Conn_01x06, J6 Conn_01x06, J7 Conn_01x06, J8 Conn_01x04, J9 Conn_01x04, SW1 SW_SPDT, SW2 SW_SPDT, SW3 SW_SPDT, SW4 SW_SPST, U1 74AUC1G19, U2 XL4015, U3 FM24W256

Commit message: Add files via upload
Parts:
- removed CC1: 1u, Capacitor_SMD:C_0603_1608Metric_Pad1.08x0.95mm_HandSolder
- removed SW1, SW2, SW3: SW_SPDT, Button_Switch_SMD:SW_SPST_Panasonic_EVQPL_3PL_5PL_PT_A15
- added C14: 10u, Capacitor_SMD:C_0805_2012Metric_Pad1.18x1.45mm_HandSolder, B.Cu at (158.2, 91.6)
- added C15: 0.1u, Capacitor_SMD:C_0603_1608Metric_Pad1.08x0.95mm_HandSolder, B.Cu at (162.9, 98.4)
- added C19: 100n, Capacitor_SMD:C_0603_1608Metric_Pad1.08x0.95mm_HandSolder, F.Cu at (170.4, 65.2)
- added C20: 100n, Capacitor_SMD:C_0603_1608Metric_Pad1.08x0.95mm_HandSolder, B.Cu at (165.2, 88.3)
- added C21: 1u, Capacitor_SMD:C_0603_1608Metric_Pad1.08x0.95mm_HandSolder, F.Cu at (160.8, 88.3)
- added C22: 10n, Capacitor_SMD:C_0603_1608Metric_Pad1.08x0.95mm_HandSolder, B.Cu at (142.3, 68.9)
- added C23: 10n, Capacitor_SMD:C_0603_1608Metric_Pad1.08x0.95mm_HandSolder, B.Cu at (142.3, 73.3)
- added Cout2: 22u, Capacitor_SMD:C_0805_2012Metric_Pad1.18x1.45mm_HandSolder, B.Cu at (162.1, 102.6)
- added D7: WS2812B-2020, LED_SMD:LED_WS2812B-2020_PLCC4_2.0x2.0mm, F.Cu at (160.7, 90.6)
- added D8: WS2812B-2020, LED_SMD:LED_WS2812B-2020_PLCC4_2.0x2.0mm, F.Cu at (164.3, 90.5)
- added J13: Conn_01x04, Connector_JST:JST_ZH_B4B-ZR_1x04_P1.50mm_Vertical, F.Cu at (175.2, 85.3)
- added J15: Conn_01x04, Connector_JST:JST_ZH_B4B-ZR_1x04_P1.50mm_Vertical, F.Cu at (155.4, 117.9)
- added J17: Conn_01x04, Connector_JST:JST_ZH_B4B-ZR_1x04_P1.50mm_Vertical, F.Cu at (171.7, 117.8)
- added R1: 100k, Resistor_SMD:R_0603_1608Metric_Pad0.98x0.95mm_HandSolder, B.Cu at (162.8, 92.5)
- added U4: TMUX1574PW, Package_SO:TSSOP-16_4.4x5mm_P0.65mm, B.Cu at (137.1, 71.2)
- C1: value 1u -> 10u; footprint Capacitor_SMD:C_0603_1608Metric_Pad1.08x0.95mm_HandSolder -> Capacitor_SMD:C_0805_2012Metric_Pad1.18x1.45mm_HandSolder
- C10, C106, C107, C108, C9: moved to B.Cu
- C101, C104, C17, Cin1: footprint Capacitor_SMD:C_0603_1608Metric_Pad1.08x0.95mm_HandSolder -> Capacitor_SMD:C_0805_2012Metric_Pad1.18x1.45mm_HandSolder
- C117: footprint Capacitor_SMD:C_0603_1608Metric_Pad1.08x0.95mm_HandSolder -> Capacitor_SMD:C_0805_2012Metric_Pad1.18x1.45mm_HandSolder; moved to F.Cu
- C18: value 1u -> 100n
- C8: value 100n -> 10n; moved to B.Cu
- Cout1: value 330u -> 22u; footprint Capacitor_SMD:C_0603_1608Metric_Pad1.08x0.95mm_HandSolder -> Capacitor_SMD:C_0805_2012Metric_Pad1.18x1.45mm_HandSolder
- D1, D2, D3: footprint LED_SMD:LED_0603_1608Metric_Pad1.05x0.95mm_HandSolder -> LED_SMD:LED_0805_2012Metric_Pad1.15x1.40mm_HandSolder; moved to F.Cu
- D101, D102: footprint Diode_SMD:D_SMA -> Diode_SMD:D_SMA_Handsoldering
- D4, D5: value D -> SS54B; footprint Diode_SMD:D_SMA_Handsoldering -> SS54B:DIOM4336X244N
- D6: value D -> WS2812B-2020; footprint Diode_SMD:D_SMA_Handsoldering -> LED_SMD:LED_WS2812B-2020_PLCC4_2.0x2.0mm; moved to F.Cu
- F1: footprint Fuse:Fuse_1210_3225Metric_Pad1.42x2.65mm_HandSolder -> Fuse:Fuse_Littelfuse-NANO2-451_453
- J1, R109, RUSB1: moved to F.Cu
- J10, J12, J14, J8, J9: footprint Connector_Hirose:Hirose_DF13-04P-1.25DSA_1x04_P1.25mm_Vertical -> Connector_JST:JST_ZH_B4B-ZR_1x04_P1.50mm_Vertical
- J11, J16: footprint Connector_Hirose:Hirose_DF13-06P-1.25DSA_1x06_P1.25mm_Vertical -> Connector_JST:JST_ZH_B6B-ZR_1x06_P1.50mm_Vertical
- J3: footprint TerminalBlock:TerminalBlock_MaiXu_MX126-5.0-02P_1x02_P5.00mm -> TerminalBlock_Phoenix:TerminalBlock_Phoenix_MPT-0,5-2-2.54_1x02_P2.54mm_Horizontal
- J4: footprint Connector_JST:JST_PH_B3B-PH-K_1x03_P2.00mm_Vertical -> Connector_JST:JST_VH_B3P-VH_1x03_P3.96mm_Vertical
- J5, J6, J7: value Conn_01x06 -> Screw_Terminal_01x02; footprint Connector_Hirose:Hirose_DF13-06P-1.25DSA_1x06_P1.25mm_Vertical -> TerminalBlock_Phoenix:TerminalBlock_Phoenix_MPT-0,5-2-2.54_1x02_P2.54mm_Horizontal
- L1: value 47u -> 3.3u; footprint Inductor_SMD:L_Bourns_SRP1245A -> Inductor_SMD:L_Bourns_SRP7028A_7.3x6.6mm
- R17, R18, R19: value 1.8k -> 330; moved to B.Cu
- R902: value 42k -> 75k
- U2: value XL4015 -> TPS565201DDCR; footprint Package_TO_SOT_SMD:TO-263-5_TabPin3 -> TPS565201DDCR:SOT95P280X110-6N
- moved J8 113.6 mm to (179.4, 104.7), turned to 180 degrees
- moved J4 112.7 mm to (176.3, 98.8), turned to 90 degrees
- moved CFF1 104.7 mm to (169.8, 97.9)
- moved R902 101.3 mm to (167.8, 102.4)
- moved R901 98.4 mm to (167.8, 93.5), turned to 90 degrees
- moved C1 90.4 mm to (155.8, 91.5), turned to 90 degrees
- moved D6 87.6 mm to (156.9, 90.6), turned to -90 degrees
- moved Cout1 85.0 mm to (165.1, 102.6)
- moved Cin1 84.6 mm to (153.4, 91.5), turned to 90 degrees
- moved L1 84.1 mm to (155.8, 100.7), turned to -90 degrees
- moved J9 82.2 mm to (179.4, 109.2)
- moved U2 80.8 mm to (162.9, 95.5)
- moved J16 73.3 mm to (153.8, 65.3), turned to 180 degrees
- moved C10 73.1 mm to (159.7, 113.4), turned to -90 degrees
- moved D5 73.0 mm to (147.3, 92.2)
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Connections:
- C10 pad 1: ADC2 -> VMOT
- C18 pad 1: +6V5 -> VMOT
- C9 pad 1: ADC1 -> VMOT
- CFF1 pad 2: Net-(U2-FB) -> Net-(U2-VFB)
- D6 pad 1: Net-(D6-K) -> Net-(D6-DOUT)
- F1 pad 2: Net-(D4-K) -> Net-(D4-PadC)
- J10 pad 3: +6V5 -> +3V3
- J11 pad 2: ADC2_EXT -> GPIO24
- J11 pad 3: ADC1_EXT -> GPIO25
- J11 pad 4: ADC0_EXT -> ADC2_EXT
- J11 pad 5: unconnected-(J11-Pin_5-Pad5) -> ADC1_EXT
- J11 pad 6: unconnected-(J11-Pin_6-Pad6) -> ADC0_EXT
- J12 pad 1: GPIO25 -> ENC0B
- J12 pad 2: GPIO24 -> ENC0A
- J12 pad 3: GPIO23 -> +3V3
- J12 pad 4: GPIO20 -> GND
- J14 pad 1: SPIO_MOSI -> EXT_nCS
- J14 pad 2: SPIO_CLK -> SPIO_MISO
- J14 pad 3: SPIO_MISO -> SPIO_CLK
- J14 pad 4: EXT_nCS -> SPIO_MOSI
- J16 pad 3: unconnected-(J16-Pin_3-Pad3) -> +3V3
- J16 pad 4: unconnected-(J16-Pin_4-Pad4) -> GND
- J2 pad 1: Net-(D4-A) -> Net-(D4-PadA)
- J3 pad 1: Net-(D5-A) -> Net-(J3-Pin_1)
- J5 pad 1: ENC0B -> M0+
- J5 pad 2: ENC0A -> M0-
- J6 pad 1: ENC1B -> M1+
- J6 pad 2: ENC1A -> M1-
- J7 pad 1: ENC2B -> M2+
- J7 pad 2: ENC2A -> M2-
- J8 pad 1: +6V5 -> +3V3
- J9 pad 3: +6V5 -> +3V3
- L1 pad 1: Net-(D6-K) -> Net-(U2-SW)
- R27 pad 1: VMOT -> BATT
- R901 pad 1: Net-(U2-FB) -> Net-(U2-VFB)
- R902 pad 2: Net-(U2-FB) -> Net-(U2-VFB)
- U2 pad 2: Net-(U2-FB) -> Net-(U2-SW)
- U2 pad 3: Net-(D6-K) -> BATT
- U2 pad 4: Net-(U2-VC) -> Net-(U2-VFB)
- U2 pad 5: BATT -> Net-(U2-EN)
- UDRV1 pad 18: GND -> (no net)
- UDRV1 pad 19: GND -> (no net)
- UDRV1 pad 20: GND -> (no net)
- UDRV1 pad 21: GND -> (no net)
- UDRV1 pad 22: GND -> (no net)
- UDRV1 pad 23: GND -> (no net)
- UDRV1 pad 24: GND -> (no net)
- UDRV1 pad 25: GND -> (no net)
- UDRV1 pad 26: GND -> (no net)
- UDRV2 pad 18: GND -> (no net)
- UDRV2 pad 19: GND -> (no net)
- UDRV2 pad 20: GND -> (no net)
- UDRV2 pad 21: GND -> (no net)
- UDRV2 pad 22: GND -> (no net)
- UDRV2 pad 23: GND -> (no net)
- UDRV2 pad 24: GND -> (no net)
- UDRV2 pad 25: GND -> (no net)
- UDRV2 pad 26: GND -> (no net)
- UDRV2 pad 27: GND -> (no net)
- UDRV2 pad 28: GND -> (no net)
- UDRV2 pad 29: GND -> (no net)
- UDRV3 pad 18: GND -> (no net)
- UDRV3 pad 19: GND -> (no net)
- UDRV3 pad 20: GND -> (no net)
- UDRV3 pad 21: GND -> (no net)
- UDRV3 pad 22: GND -> (no net)
- UDRV3 pad 23: GND -> (no net)
- UDRV3 pad 24: GND -> (no net)
- UDRV3 pad 25: GND -> (no net)
- UDRV3 pad 26: GND -> (no net)
- UDRV3 pad 27: GND -> (no net)
- UDRV3 pad 28: GND -> (no net)
- UDRV3 pad 29: GND -> (no net)
- URP2040 pad 35: GPIO23 -> MUX_S0
Routing:
- net GND: track 337.6 -> 0.00 mm, vias 67 -> 0
- net +6V5: track 138.5 -> 0.00 mm, vias 10 -> 0
- net VMOT: track 126.4 -> 0.00 mm, vias 13 -> 0
- net +3V3: track 132.0 -> 20.9 mm, vias 39 -> 4
- net ADC1: track 73.8 -> 9.40 mm, vias 3 -> 1
- net ADC2: track 69.8 -> 7.70 mm, vias 3 -> 1
- net M0_DIR: track 61.5 -> 1.64 mm, vias 2 -> 1
- net M0_PWM: track 57.1 -> 0.00 mm, vias 1 -> 0
- net ENC0A: track 52.5 -> 0.00 mm, vias 1 -> 0
- net M1_DIR: track 53.0 -> 1.18 mm, vias 2 -> 1
- net ENC0B: track 51.0 -> 0.00 mm, vias 1 -> 0
- net M2_DIR: track 49.2 -> 1.26 mm, vias 2 -> 1
- net M1_PWM: track 45.8 -> 0.00 mm, vias 1 -> 0
- net ENC1A: track 45.7 -> 0.00 mm, vias 1 -> 0
- net ENC1B: track 45.4 -> 0.00 mm, vias 1 -> 0
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- added copper zone on F.Cu, net GND
- removed copper zone on F.Cu, net +3V3
- removed copper zone on In2.Cu, net +6V5
- removed copper zone on In2.Cu, net BATT
- removed copper zone on In1.Cu, net GND
- removed copper zone on In2.Cu, net VMOT
Other:
- outline, holes or cut-outs redrawn
- board text added: "100uF"
- board text added: "10k"
- board text added: "1k"
- board text added: "220n"
- board text removed: "+"
- board text removed: "0"
- board text removed: "0A"
- board text removed: "0B"
- board text removed: "1"
- board text removed: "10K"
- board text removed: "10uF"
- board text removed: "15pF"
- board text removed: "1A"
- board text removed: "1B"
- board text removed: "1K"
- board text removed: "1uF"
- board text removed: "2"
- board text removed: "2.2nF"
- board text removed: "20"
- board text removed: "220uF"
- board text removed: "23"
- board text removed: "24"
- board text removed: "25"
- board text removed: "27 OHM"
- board text removed: "2A"
- board text removed: "2B"
- board text removed: "3.3V"
- board text removed: "330uF"
- board text removed: "33nF"
- board text removed: "4.7K"
- board text removed: "42K"
- board text removed: "47K"
- board text removed: "47uH / 5A"
- board text removed: "5.1K"
- board text removed: "5A"
- board text removed: "6.5V"
- board text removed: "74AUC1G19"
- board text removed: "ADC EXT"
- board text removed: "ADC0"
- board text removed: "ADC1"
- board text removed: "ADC2"
- board text removed: "Barrel Jack"
- board text removed: "DIR"
- board text removed: "ENC"
- board text removed: "ESD"
- board text removed: "FB"
- board text removed: "FRAM"
- board text removed: "FUSE"
- board text removed: "Flash Memory"
- board text removed: "GND"
- board text removed: "GPIO"
- board text removed: "LED"
- board text removed: "M0"
- board text removed: "M0+"
- board text removed: "M0-"
- board text removed: "M1"
- board text removed: "M1+"
- board text removed: "M1-"
- board text removed: "M2"
- board text removed: "M2+"
- board text removed: "M2-"
- board text removed: "MOSI | CLK | MISO | CS"
- board text removed: "MOTOR"
- board text removed: "NCP1117"
- board text removed: "PWM"
- board text removed: "RAW"
- board text removed: "RESET"
- board text removed: "RUN"
- board text removed: "SPIO"
- board text removed: "SS14"
- board text removed: "SS54"
- board text removed: "Screw Terminal"
- board text removed: "UART RX"
- board text removed: "UART TX"
- board text removed: "USBC"
- board text removed: "XL4015"
