File: LDO.kicad_sch (KiCad schematic)
At the start: 3 parts, among them U4 AMS1117-5.0

Commit message: Add files via upload
Parts:
- removed C14, C15: 22u, Capacitor_SMD:C_2220_5750Metric_Pad1.97x5.40mm_HandSolder, symbol Device:C
- removed U4: AMS1117-5.0, Package_TO_SOT_SMD:SOT-223-3_TabPin2, symbol Regulator_Linear:AMS1117-5.0
