File: CurrentSensing.kicad_sch (KiCad schematic)
At the start: 9 parts, among them SW1 SW_SPDT, SW2 SW_SPDT, SW3 SW_SPDT

Commit message: Add files via upload
Parts:
- C10, C8, C9: footprint Capacitor_SMD:C_2220_5750Metric_Pad1.97x5.40mm_HandSolder -> Capacitor_SMD:C_0603_1608Metric_Pad1.08x0.95mm_HandSolder
- R17, R18, R19: footprint Resistor_SMD:R_2010_5025Metric_Pad1.40x2.65mm_HandSolder -> Resistor_SMD:R_0603_1608Metric_Pad0.98x0.95mm_HandSolder
- SW1, SW2, SW3: footprint Button_Switch_SMD:SW_Push_1P1T-SH_NO_CK_KMR2xxG -> Button_Switch_SMD:SW_SPST_Panasonic_EVQPL_3PL_5PL_PT_A15
Changed lines of the file:
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@@
 	(wire
 		(pts
-			(xy 160.02 63.5) (xy 154.94 63.5)
+			(xy 168.91 63.5) (xy 154.94 63.5)
 		)
 		(stroke
@@
 	(wire
 		(pts
+			(xy 121.92 123.19) (xy 140.97 123.19)
+		)
+		(stroke
+			(width 0)
+			(type default)
+		)
+	)
+	(wire
+		(pts
+			(xy 160.02 92.71) (xy 154.94 92.71)
+		)
+		(stroke
+			(width 0)
+			(type default)
+		)
+	)
+	(wire
+		(pts
+			(xy 154.94 123.19) (xy 148.59 123.19)
+		)
+		(stroke
+			(width 0)
+			(type default)
+		)
+	)
+	(wire
+		(pts
 			(xy 121.92 109.22) (xy 121.92 123.19)
-		)
-		(stroke
-			(width 0)
-			(type default)
-		)
-	)
-	(wire
-		(pts
-			(xy 121.92 123.19) (xy 140.97 123.19)
-		)
-		(stroke
-			(width 0)
-			(type default)
-		)
-	)
-	(wire
-		(pts
-			(xy 160.02 92.71) (xy 154.94 92.71)
-		)
-		(stroke
-			(width 0)
-			(type default)
-		)
-	)
-	(wire
-		(pts
-			(xy 154.94 123.19) (xy 148.59 123.19)
 		)
 		(stroke
@@
 		)
 	)
+	(global_label "ADC0_EXT"
+		(shape input)
+		(at 87.63 80.01 180)
+		(fields_autoplaced yes)
+		(effects
+			(font
+				(size 1.27 1.27)
+			)
+			(justify right)
+		)
+		(property "Intersheetrefs" "${INTERSHEET_REFS}"
+			(at 75.513 80.01 0)
+			(effects
+				(font
+					(size 1.27 1.27)
+				)
+				(justify right)
+				(hide yes)
+			)
+		)
+	)
 	(global_label "ADC2"
 		(shape input)
@@
 	(global_label "ADC0"
 		(shape input)
-		(at 160.02 63.5 0)
+		(at 168.91 63.5 0)
 		(fields_autoplaced yes)
 		(effects
@@
 		)
 		(property "Intersheetrefs" "${INTERSHEET_REFS}"
-			(at 167.8433 63.5 0)
+			(at 176.7333 63.5 0)
 			(effects
 				(font
@@
 				)
 				(justify left)
-				(hide yes)
-			)
-		)
-	)
-	(global_label "ADC0_EXT"
-		(shape input)
-		(at 87.63 80.01 180)
-		(fields_autoplaced yes)
-		(effects
-			(font
-				(size 1.27 1.27)
-			)
-			(justify right)
-		)
-		(property "Intersheetrefs" "${INTERSHEET_REFS}"
-			(at 75.513 80.01 0)
-			(effects
-				(font
-					(size 1.27 1.27)
-				)
-				(justify right)
 				(hide yes)
 			)
@@
 			)
 		)
-		(property "Footprint" "Capacitor_SMD:C_2220_5750Metric_Pad1.97x5.40mm_HandSolder"
+		(property "Footprint" "Capacitor_SMD:C_0603_1608Metric_Pad1.08x0.95mm_HandSolder"
 			(at 153.9748 104.14 0)
 			(effects
@@
 			)
 		)
-		(property "Footprint" "Button_Switch_SMD:SW_Push_1P1T-SH_NO_CK_KMR2xxG"
+		(property "Footprint" "Button_Switch_SMD:SW_SPST_Panasonic_EVQPL_3PL_5PL_PT_A15"
 			(at 101.6 92.71 0)
 			(effects
@@
 			)
 		)
-		(property "Footprint" "Resistor_SMD:R_2010_5025Metric_Pad1.40x2.65mm_HandSolder"
+		(property "Footprint" "Resistor_SMD:R_0603_1608Metric_Pad0.98x0.95mm_HandSolder"
 			(at 144.78 94.488 90)
 			(effects
@@
 			)
 		)
-		(property "Footprint" "Capacitor_SMD:C_2220_5750Metric_Pad1.97x5.40mm_HandSolder"
+		(property "Footprint" "Capacitor_SMD:C_0603_1608Metric_Pad1.08x0.95mm_HandSolder"
 			(at 153.9748 134.62 0)
 			(effects
@@
 			)
 		)
-		(property "Footprint" "Resistor_SMD:R_2010_5025Metric_Pad1.40x2.65mm_HandSolder"
+		(property "Footprint" "Resistor_SMD:R_0603_1608Metric_Pad0.98x0.95mm_HandSolder"
 			(at 144.78 124.968 90)
 			(effects
@@
 			)
 		)
-		(property "Footprint" "Capacitor_SMD:C_2220_5750Metric_Pad1.97x5.40mm_HandSolder"
+		(property "Footprint" "Capacitor_SMD:C_0603_1608Metric_Pad1.08x0.95mm_HandSolder"
 			(at 153.9748 74.93 0)
 			(effects
@@
 			)
 		)
-		(property "Footprint" "Button_Switch_SMD:SW_Push_1P1T-SH_NO_CK_KMR2xxG"
+		(property "Footprint" "Button_Switch_SMD:SW_SPST_Panasonic_EVQPL_3PL_5PL_PT_A15"
 			(at 101.6 77.47 0)
 			(effects
@@
 			)
 		)
-		(property "Footprint" "Button_Switch_SMD:SW_Push_1P1T-SH_NO_CK_KMR2xxG"
+		(property "Footprint" "Button_Switch_SMD:SW_SPST_Panasonic_EVQPL_3PL_5PL_PT_A15"
 			(at 101.6 109.22 0)
 			(effects
@@
 			)
 		)
-		(property "Footprint" "Resistor_SMD:R_2010_5025Metric_Pad1.40x2.65mm_HandSolder"
+		(property "Footprint" "Resistor_SMD:R_0603_1608Metric_Pad0.98x0.95mm_HandSolder"
 			(at 144.78 65.278 90)
 			(effects

Commit message: Add files via upload
Parts:
- removed C10, C9: 100n, Capacitor_SMD:C_0603_1608Metric_Pad1.08x0.95mm_HandSolder, symbol Device:C
- removed SW1, SW2, SW3: SW_SPDT, Button_Switch_SMD:SW_SPST_Panasonic_EVQPL_3PL_5PL_PT_A15, symbol Switch:SW_SPDT
- added C22, C23: 10n, Capacitor_SMD:C_0603_1608Metric_Pad1.08x0.95mm_HandSolder, symbol Device:C
- added U4: TMUX1574PW, Package_SO:TSSOP-16_4.4x5mm_P0.65mm, symbol Analog_Switch:TMUX1574PW
- C8: value 100n -> 10n
- R17, R18, R19: value 1.8k -> 330
Connections:
- net ADC0_EXT: now also U4.3 (S1B)
- net ADC1: now also C22.1
- net ADC1_EXT: now also U4.6 (S2B)
- net ADC2: now also C23.1
- net ADC2_EXT: now also U4.10 (S3B)
- net GND: now also C22.2, C23.2, U4.13 (S4B), U4.14 (S4A), U4.15 (~{EN}), U4.8 (GND)
- net M0_CS: now also U4.2 (S1A)
- net M1_CS: now also U4.5 (S2A)
- net M2_CS: now also U4.11 (S3A)
- net at R18.2: now also U4.7 (D2)
- net at R19.2: now also U4.9 (D3)
- net at R17.2: now also U4.4 (D1)
- new net +3V3: U4.16 (VDD)
- new net MUX_S0: U4.1 (SEL)
- no-connect marks 0 -> 1
Other:
- note added: "Quad 2:1 Multiplexer Code controlled to read Current sensing values or analog values from externally connected sensors"
- moved on the sheet: C8, R17
