File: FRAM.kicad_sch (KiCad schematic)
At the start: 1 part, among them U3 FM24W256

Commit message: Add files via upload
Other:
- note added: "Current address 0x50 Supports 100 trillion writes"
Changed lines of the file:
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@@
 		(company "Astra Robotics")
+	)
+	(rectangle
+		(start 96.52 55.88)
+		(end 146.05 99.06)
+		(stroke
+			(width 0)
+			(type solid)
+		)
+		(fill
+			(type none)
+		)
+	)
+	(text "Current address 0x50\nSupports 100 trillion writes\n"
+		(exclude_from_sim no)
+		(at 122.174 91.694 0)
+		(effects
+			(font
+				(size 1.27 1.27)
+			)
+		)
 	)
 	(junction
