File: MotorVoltageSelectJumper.kicad_sch (KiCad schematic)
At the start: 1 part, among them J4 Conn_01x03

Commit message: Add files via upload
Parts:
- J4: footprint Connector:FanPinHeader_1x03_P2.54mm_Vertical -> Connector_JST:JST_PH_B3B-PH-K_1x03_P2.00mm_Vertical
Changed lines of the file:
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@@
 			)
 		)
-		(property "Footprint" "Connector:FanPinHeader_1x03_P2.54mm_Vertical"
+		(property "Footprint" "Connector_JST:JST_PH_B3B-PH-K_1x03_P2.00mm_Vertical"
 			(at 127 106.68 0)
 			(effects

Commit message: Add files via upload
Parts:
- J4: footprint Connector_JST:JST_PH_B3B-PH-K_1x03_P2.00mm_Vertical -> Connector_JST:JST_VH_B3P-VH_1x03_P3.96mm_Vertical
Other:
- note added: "Will be a shorting jumper Shorting 2 & 1 provides raw unregulated power Shorting 2 & 3 provides regulated constant 6.5V"
Changed lines of the file:
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@@
 		(company "Astra Robotics")
+	)
+	(rectangle
+		(start 93.98 87.63)
+		(end 146.05 124.46)
+		(stroke
+			(width 0)
+			(type solid)
+			(color 0 0 0 1)
+		)
+		(fill
+			(type none)
+		)
+	)
+	(text "Will be a shorting jumper \nShorting 2 & 1 provides raw unregulated power \nShorting 2 & 3 provides regulated constant 6.5V "
+		(exclude_from_sim no)
+		(at 121.158 117.856 0)
+		(effects
+			(font
+				(size 1.27 1.27)
+			)
+		)
 	)
 	(wire
@@
 			)
 		)
-		(property "Footprint" "Connector_JST:JST_PH_B3B-PH-K_1x03_P2.00mm_Vertical"
+		(property "Footprint" "Connector_JST:JST_VH_B3P-VH_1x03_P3.96mm_Vertical"
 			(at 127 106.68 0)
 			(effects
