File: RP2040.kicad_sch (KiCad schematic)
At the start: 37 parts, among them SW4 SW_SPST

Commit message: Add files via upload
Parts:
- C101, C104, C117: footprint Capacitor_SMD:C_0603_1608Metric_Pad1.08x0.95mm_HandSolder -> Capacitor_SMD:C_0805_2012Metric_Pad1.18x1.45mm_HandSolder
- D101, D102: footprint Diode_SMD:D_SMA -> Diode_SMD:D_SMA_Handsoldering
Connections:
- net GPIO23 renamed MUX_S0
Changed lines of the file:
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@@
 		)
 	)
-	(global_label "GPIO24"
+	(global_label "SWCLK"
 		(shape input)
-		(at 226.06 147.32 0)
+		(at 195.58 157.48 0)
 		(fields_autoplaced yes)
 		(effects
@@
 		)
 		(property "Intersheetrefs" "${INTERSHEET_REFS}"
-			(at 235.9395 147.32 0)
+			(at 204.7942 157.48 0)
 			(effects
 				(font
@@
 		)
 	)
-	(global_label "SWCLK"
+	(global_label "SPIO_CS"
 		(shape input)
-		(at 195.58 157.48 0)
+		(at 266.7 153.67 0)
 		(fields_autoplaced yes)
 		(effects
@@
 		)
 		(property "Intersheetrefs" "${INTERSHEET_REFS}"
-			(at 204.7942 157.48 0)
+			(at 277.5471 153.67 0)
 			(effects
 				(font
@@
 		)
 	)
-	(global_label "GPIO25"
+	(global_label "UART0_RX"
 		(shape input)
-		(at 226.06 151.13 0)
+		(at 269.24 49.53 0)
 		(fields_autoplaced yes)
 		(effects
@@
 		)
 		(property "Intersheetrefs" "${INTERSHEET_REFS}"
-			(at 235.9395 151.13 0)
+			(at 281.5385 49.53 0)
 			(effects
 				(font
@@
 		)
 	)
-	(global_label "SPIO_CS"
+	(global_label "GPIO24"
 		(shape input)
-		(at 266.7 153.67 0)
+		(at 226.06 147.32 0)
 		(fields_autoplaced yes)
 		(effects
@@
 		)
 		(property "Intersheetrefs" "${INTERSHEET_REFS}"
-			(at 277.5471 153.67 0)
+			(at 235.9395 147.32 0)
 			(effects
 				(font
@@
 		)
 	)
-	(global_label "UART0_RX"
+	(global_label "ADC0"
 		(shape input)
-		(at 269.24 49.53 0)
+		(at 271.78 86.36 0)
 		(fields_autoplaced yes)
 		(effects
@@
 		)
 		(property "Intersheetrefs" "${INTERSHEET_REFS}"
-			(at 281.5385 49.53 0)
+			(at 279.6033 86.36 0)
 			(effects
 				(font
@@
 		)
 	)
-	(global_label "ADC0"
+	(global_label "M2_DIR"
 		(shape input)
-		(at 271.78 86.36 0)
+		(at 270.51 78.74 0)
 		(fields_autoplaced yes)
 		(effects
@@
 		)
 		(property "Intersheetrefs" "${INTERSHEET_REFS}"
-			(at 279.6033 86.36 0)
+			(at 280.2685 78.74 0)
 			(effects
 				(font
@@
 		)
 	)
-	(global_label "M2_DIR"
+	(global_label "ENC1B"
 		(shape input)
-		(at 270.51 78.74 0)
+		(at 270.51 135.89 0)
 		(fields_autoplaced yes)
 		(effects
@@
 		)
 		(property "Intersheetrefs" "${INTERSHEET_REFS}"
-			(at 280.2685 78.74 0)
+			(at 279.7242 135.89 0)
 			(effects
 				(font
@@
 		)
 	)
-	(global_label "ENC1B"
+	(global_label "M0_DIR"
 		(shape input)
-		(at 270.51 135.89 0)
+		(at 270.51 63.5 0)
 		(fields_autoplaced yes)
 		(effects
@@
 		)
 		(property "Intersheetrefs" "${INTERSHEET_REFS}"
-			(at 279.7242 135.89 0)
+			(at 280.2685 63.5 0)
 			(effects
 				(font
@@
 		)
 	)
-	(global_label "M0_DIR"
+	(global_label "GPIO25"
 		(shape input)
-		(at 270.51 63.5 0)
+		(at 226.06 151.13 0)
 		(fields_autoplaced yes)
 		(effects
@@
 		)
 		(property "Intersheetrefs" "${INTERSHEET_REFS}"
-			(at 280.2685 63.5 0)
+			(at 235.9395 151.13 0)
 			(effects
 				(font
@@
 		)
 	)
-	(global_label "SPIO_MISO"
+	(global_label "MUX_S0"
 		(shape input)
-		(at 266.7 149.86 0)
+		(at 226.06 143.51 0)
 		(fields_autoplaced yes)
 		(effects
@@
 		)
 		(property "Intersheetrefs" "${INTERSHEET_REFS}"
-			(at 279.6638 149.86 0)
+			(at 236.4232 143.51 0)
 			(effects
 				(font
@@
 		)
 	)
-	(global_label "SPIO_MOSI"
+	(global_label "SPIO_MISO"
 		(shape input)
-		(at 266.7 161.29 0)
+		(at 266.7 149.86 0)
 		(fields_autoplaced yes)
 		(effects
@@
 		)
 		(property "Intersheetrefs" "${INTERSHEET_REFS}"
-			(at 279.6638 161.29 0)
+			(at 279.6638 149.86 0)
 			(effects
 				(font
@@
 		)
 	)
-	(global_label "ENC2B"
+	(global_label "SPIO_MOSI"
 		(shape input)
-		(at 270.51 143.51 0)
+		(at 266.7 161.29 0)
 		(fields_autoplaced yes)
 		(effects
@@
 		)
 		(property "Intersheetrefs" "${INTERSHEET_REFS}"
-			(at 279.7242 143.51 0)
+			(at 279.6638 161.29 0)
 			(effects
 				(font
@@
 		)
 	)
-	(global_label "SDA"
+	(global_label "ENC2B"
 		(shape input)
-		(at 273.05 104.14 0)
+		(at 270.51 143.51 0)
 		(fields_autoplaced yes)
 		(effects
@@
 		)
 		(property "Intersheetrefs" "${INTERSHEET_REFS}"
-			(at 279.6033 104.14 0)
+			(at 279.7242 143.51 0)
 			(effects
 				(font
@@
 		)
 	)
-	(global_label "ENC0B"
+	(global_label "SDA"
 		(shape input)
-		(at 270.51 128.27 0)
+		(at 273.05 104.14 0)
 		(fields_autoplaced yes)
 		(effects
@@
 		)
 		(property "Intersheetrefs" "${INTERSHEET_REFS}"
-			(at 279.7242 128.27 0)
+			(at 279.6033 104.14 0)
 			(effects
 				(font
@@
 		)
 	)
-	(global_label "SWDIO"
+	(global_label "ENC0B"
 		(shape input)
-		(at 195.58 161.29 0)
+		(at 270.51 128.27 0)
 		(fields_autoplaced yes)
 		(effects
@@
 		)
 		(property "Intersheetrefs" "${INTERSHEET_REFS}"
-			(at 204.4314 161.29 0)
+			(at 279.7242 128.27 0)
 			(effects
 				(font
@@
 		)
 	)
-	(global_label "GPIO23"
+	(global_label "SWDIO"
 		(shape input)
-		(at 226.06 143.51 0)
+		(at 195.58 161.29 0)
 		(fields_autoplaced yes)
 		(effects
@@
 		)
 		(property "Intersheetrefs" "${INTERSHEET_REFS}"
-			(at 235.9395 143.51 0)
+			(at 204.4314 161.29 0)
 			(effects
 				(font
@@
 	)
 	(symbol
+		(lib_id "power:VBUS")
+		(at 95.25 58.42 0)
+		(unit 1)
+		(exclude_from_sim no)
+		(in_bom yes)
+		(on_board yes)
+		(dnp no)
+		(fields_autoplaced yes)
+		(property "Reference" "#PWR062"
+			(at 95.25 62.23 0)
+			(effects
+				(font
+					(size 1.27 1.27)
+				)
+				(hide yes)
+			)
+		)
+		(property "Value" "VBUS"
+			(at 95.25 53.34 0)
+			(effects
+				(font
+					(size 1.27 1.27)
+				)
+			)
+		)
+		(property "Footprint" ""
+			(at 95.25 58.42 0)
+			(effects
+				(font
+					(size 1.27 1.27)
+				)
+				(hide yes)
+			)
+		)
+		(property "Datasheet" ""
+			(at 95.25 58.42 0)
+			(effects
+				(font
+					(size 1.27 1.27)
+				)
+				(hide yes)
+			)
+		)
+		(property "Description" "Power symbol creates a global label with name \"VBUS\""
+			(at 95.25 58.42 0)
+			(effects
+				(font
+					(size 1.27 1.27)
+				)
+				(hide yes)
+			)
+		)
+		(pin "1"
+		)
+		(instances
+			(project "MBot"
+				(path "/6379cb09-8427-484b-8caa-23471c63c9c8/fba4b5c3-a0b5-43e7-8123-1a188b00f5ab"
+					(reference "#PWR062")
+					(unit 1)
+				)
+			)
+		)
+	)
+	(symbol
 		(lib_id "power:GND")
 		(at 67.31 163.83 0)
@@
 			)
 		)
-		(property "Footprint" "Capacitor_SMD:C_0603_1608Metric_Pad1.08x0.95mm_HandSolder"
+		(property "Footprint" "Capacitor_SMD:C_0805_2012Metric_Pad1.18x1.45mm_HandSolder"
 			(at 84.7852 39.37 0)
 			(effects
@@
 			)
 		)
-		(property "Footprint" "Diode_SMD:D_SMA"
+		(property "Footprint" "Diode_SMD:D_SMA_Handsoldering"
 			(at 79.375 24.13 0)
 			(effects
@@
 			)
 		)
-		(property "Footprint" "Capacitor_SMD:C_0603_1608Metric_Pad1.08x0.95mm_HandSolder"
+		(property "Footprint" "Capacitor_SMD:C_0805_2012Metric_Pad1.18x1.45mm_HandSolder"
 			(at 108.9152 39.37 0)
 			(effects
@@
 	)
 	(symbol
-		(lib_id "power:VBUS")
-		(at 95.25 58.42 0)
-		(unit 1)
-		(exclude_from_sim no)
-		(in_bom yes)
-		(on_board yes)
-		(dnp no)
-		(fields_autoplaced yes)
-		(property "Reference" "#PWR062"
-			(at 95.25 62.23 0)
-			(effects
-				(font
-					(size 1.27 1.27)
-				)
-				(hide yes)
-			)
-		)
-		(property "Value" "VBUS"
-			(at 95.25 53.34 0)
-			(effects
-				(font
-					(size 1.27 1.27)
-				)
-			)
-		)
-		(property "Footprint" ""
-			(at 95.25 58.42 0)
-			(effects
-				(font
-					(size 1.27 1.27)
-				)
-				(hide yes)
-			)
-		)
-		(property "Datasheet" ""
-			(at 95.25 58.42 0)
-			(effects
-				(font
-					(size 1.27 1.27)
-				)
-				(hide yes)
-			)
-		)
-		(property "Description" "Power symbol creates a global label with name \"VBUS\""
-			(at 95.25 58.42 0)
-			(effects
-				(font
-					(size 1.27 1.27)
-				)
-				(hide yes)
-			)
-		)
-		(pin "1"
-		)
-		(instances
-			(project "MBot"
-				(path "/6379cb09-8427-484b-8caa-23471c63c9c8/fba4b5c3-a0b5-43e7-8123-1a188b00f5ab"
-					(reference "#PWR062")
-					(unit 1)
-				)
-			)
-		)
-	)
-	(symbol
 		(lib_id "Diode:SS14")
 		(at 68.58 29.21 180)
@@
 			)
 		)
-		(property "Footprint" "Diode_SMD:D_SMA"
+		(property "Footprint" "Diode_SMD:D_SMA_Handsoldering"
 			(at 68.58 24.765 0)
 			(effects
@@
 			)
 		)
-		(property "Footprint" "Capacitor_SMD:C_0603_1608Metric_Pad1.08x0.95mm_HandSolder"
+		(property "Footprint" "Capacitor_SMD:C_0805_2012Metric_Pad1.18x1.45mm_HandSolder"
 			(at 162.2552 180.34 0)
 			(effects
