File: SwitchingRegulator.kicad_sch (KiCad schematic)
At the start: 16 parts, among them J2 Barrel_Jack_Switch_Pin3Ring, J3 Screw_Terminal_01x02, U2 XL4015

Commit message: Add files via upload
Parts:
- removed D4, D5, D6: SS54FSH, SS54FSH:SODFL4725X110N, symbol SS54FSH:SS54FSH
- added D4, D5, D6: D, Diode_SMD:D_SMA_Handsoldering, symbol Device:D
- C1: footprint (none) -> Capacitor_SMD:C_0603_1608Metric_Pad1.08x0.95mm_HandSolder
- C18, CC1, CFF1, Cin1, Cout1: footprint Capacitor_SMD:C_2220_5750Metric_Pad1.97x5.40mm_HandSolder -> Capacitor_SMD:C_0603_1608Metric_Pad1.08x0.95mm_HandSolder
- L1: footprint Inductor_SMD:L_12x12mm_H8mm -> Inductor_SMD:L_Bourns_SRP1245A
- R901, R902: footprint Resistor_SMD:R_1812_4532Metric_Pad1.30x3.40mm_HandSolder -> Resistor_SMD:R_0603_1608Metric_Pad0.98x0.95mm_HandSolder
Connections:
- net GND: now also D6.2 (A)
- net at J3.1 (Pin_1): now also D5.2 (A)
- net at F1.2: now also D4.1 (K), D5.1 (K)
- net at L1.1, U2.3 (SW): now also D6.1 (K)
- net at J2.1: now also D4.2 (A)
Other:
- moved on the sheet: C18

Commit message: Add files via upload
Parts:
- removed CC1: 1u, Capacitor_SMD:C_0603_1608Metric_Pad1.08x0.95mm_HandSolder, symbol Device:C
- removed D4, D5, D6: D, Diode_SMD:D_SMA_Handsoldering, symbol Device:D
- removed U2: XL4015, Package_TO_SOT_SMD:TO-263-5_TabPin3, symbol Regulator_Switching:XL4015
- added C14: 10u, Capacitor_SMD:C_0805_2012Metric_Pad1.18x1.45mm_HandSolder, symbol Device:C
- added C15: 0.1u, Capacitor_SMD:C_0603_1608Metric_Pad1.08x0.95mm_HandSolder, symbol Device:C
- added D4, D5: SS54B, SS54B:DIOM4336X244N, symbol SS54B:SS54B
- added R1: 100k, Resistor_SMD:R_0603_1608Metric_Pad0.98x0.95mm_HandSolder, symbol Device:R
- added U2: TPS565201DDCR, TPS565201DDCR:SOT95P280X110-6N, symbol TPS565201DDCR:TPS565201DDCR
- C1: value 1u -> 10u; footprint Capacitor_SMD:C_0603_1608Metric_Pad1.08x0.95mm_HandSolder -> Capacitor_SMD:C_0805_2012Metric_Pad1.18x1.45mm_HandSolder
- Cin1: footprint Capacitor_SMD:C_0603_1608Metric_Pad1.08x0.95mm_HandSolder -> Capacitor_SMD:C_0805_2012Metric_Pad1.18x1.45mm_HandSolder
- Cout1: value 330u -> 22u; footprint Capacitor_SMD:C_0603_1608Metric_Pad1.08x0.95mm_HandSolder -> Capacitor_SMD:C_0805_2012Metric_Pad1.18x1.45mm_HandSolder
- Cout2: renamed from C18; value 1u -> 22u; footprint Capacitor_SMD:C_0603_1608Metric_Pad1.08x0.95mm_HandSolder -> Capacitor_SMD:C_0805_2012Metric_Pad1.18x1.45mm_HandSolder
- F1: footprint Fuse:Fuse_1210_3225Metric_Pad1.42x2.65mm_HandSolder -> Fuse:Fuse_Littelfuse-NANO2-451_453
- J3: footprint TerminalBlock:TerminalBlock_MaiXu_MX126-5.0-02P_1x02_P5.00mm -> TerminalBlock_Phoenix:TerminalBlock_Phoenix_MPT-0,5-2-2.54_1x02_P2.54mm_Horizontal
- L1: value 47u -> 3.3u; footprint Inductor_SMD:L_Bourns_SRP1245A -> Inductor_SMD:L_Bourns_SRP7028A_7.3x6.6mm
- R902: value 42k -> 75k
Connections:
- net BATT: now also C14.1, R1.1, U2.3 (VIN)
- net GND: now also C14.2, U2.1 (GND)
- net at F1.2: now also D4.C, D5.C
- net at J3.1 (Pin_1): now also D5.A
- net at CFF1.2, R901.1, R902.2: now also U2.4 (VFB)
- net at L1.1: now also C15.1, U2.2 (SW)
- net at J2.1: now also D4.A
- new net: R1.2, U2.5 (EN)
- new net: C15.2, U2.6 (VBST)
Other:
- note added: "3.3u/5A"
- note added: "Ceramic"
- note added: "Electrolytic"
- note added: "TPS565201 Synchronous Step-Down"
- note removed: "330uF/25V"
- note removed: "47uH/5A"
- moved on the sheet: C1, Cin1
